Commit message: Backup commit

File: my_robot/urdf/my_robot.xacro (robot description, xacro)
@@ -158,5 +158,5 @@
     	<axis xyz="0 1 0" rpy="0 0 0"/>
     </joint>
-  <link name='camera'>
+  <link name='camera_link'>
     <visual name='camera_visual'>
       <origin xyz="0 0 0" rpy=" 0 0 0"/>
@@ -183,8 +183,15 @@
   <joint type="fixed" name="camera_joint">
     <origin xyz="-0.15 0 0.145" rpy="0 0 3.1415"/>
-    <child link="camera"/>
+    <child link="camera_link"/>
     <parent link="chassis"/>
     <axis xyz="0 1 0" rpy="0 0 0"/>
   </joint>
+  <joint name="camera_optical_joint" type="fixed">
+    <origin xyz="0 0 0" rpy="-1.5707 0 -1.5707"/>
+    <parent link="camera_link"/>
+    <child link="camera_link_optical"/>
+  </joint>
+  <link name="camera_link_optical">
+  </link>
   <gazebo reference="camera">
     <material>Gazebo/Black</material>

Commit message: Removed oversized file and added db file link

File: my_robot/urdf/my_robot.xacro (robot description, xacro)
@@ -103,5 +103,5 @@
   <link name='hokuyo'>
     <visual name='hokuyo_visual'>
-    <origin xyz="0 0 0" rpy=" 0 0 0"/>
+    <origin xyz="0 0 0" rpy=" 0 0 3.14"/>
       <geometry>
         <mesh filename="package://my_robot/meshes/hokuyo.dae"/>
@@ -109,5 +109,5 @@
     </visual>
     <collision name='hokuyo_collision'>
-      <origin xyz="0 0 0" rpy=" 0 0 0"/>
+      <origin xyz="0 0 0" rpy=" 0 0 3.14"/>
       <geometry>
         <box size=".1 .1 .1"/>
@@ -116,5 +116,5 @@
     <inertial>
       <mass value="1e-5"/>
-      <origin xyz="0 0 0" rpy=" 0 0 0 "/>
+      <origin xyz="0 0 0" rpy=" 0 0 3.14 "/>
       <inertia
          ixx="1e-6" ixy="0" ixz="0"
@@ -124,5 +124,5 @@
    </link>
     <joint type="fixed" name="hokuyo_joint">
-    	<origin xyz="0 0 0.16" rpy="0 0 0"/>
+    	<origin xyz="0 0 0.16" rpy="0 0 3.14"/>
    	  <child link="hokuyo"/>
     	<parent link="chassis"/>
